Commit message: Integrated Lidar with the Robot

File: src/my_bot/description/robot.urdf.xacro (robot description, xacro)
@@ -4,3 +4,4 @@
     <xacro:include filename="robot_core.xacro" />
     <xacro:include filename="gazebo_control.xacro"/>
+    <xacro:include filename="lidar.xacro"/>
 </robot>

File: src/my_bot/description/robot_core.xacro (robot description, xacro)
@@ -13,4 +13,7 @@
     <material name="blue">
         <color rgba="0 0 1 1"/>
+    </material>
+    <material name="red">
+        <color rgba="1 0 0 1"/>
     </material>
     <!-- Base Link  -->
